Commit message: fixed files names clean the urdf description

File: spcbot_description/urdf/spcbot.gazebo.xacro (robot description, xacro)
@@ -1,8 +1,9 @@
 <?xml version='1.0'?>
-<robot>
-  <gazebo reference="camera">
+<robot name="spcbot_gazebo" xmlns:xacro="http://ros.org/wiki/xacro">
+  <gazebo reference="camera_link">
     <material>Gazebo/Green</material>
-    <sensor type="camera" name="camera1">
+    <sensor type="camera" name="camera">
       <update_rate>30.0</update_rate>
+      <visualize></visualize>
       <camera name="head">
         <horizontal_fov>1.3962634</horizontal_fov>
@@ -20,5 +21,5 @@
         <alwaysOn>true</alwaysOn>
         <updateRate>0.0</updateRate>
-        <cameraName>spcbot/camera1</cameraName>
+        <cameraName>spcbot/camera</cameraName>
         <imageTopicName>image_raw</imageTopicName>
         <cameraInfoTopicName>camera_info</cameraInfoTopicName>

File: spcbot_description/urdf/spcbot.urdf.xacro (robot description, xacro)
@@ -4,9 +4,9 @@
   <xacro:property name="cameraMass" value="0.1"/>
   <xacro:include filename="$(find spcbot_description)/urdf/materials.xacro"/>
-  <xacro:include filename="$(find spcbot_description)/urdf/spcbot.gazebo"/>
+  <xacro:include filename="$(find spcbot_description)/urdf/spcbot.gazebo.xacro"/>
   <link name='chassis'>
     <pose>0 0 0.1 0 0 0</pose>
     <inertial>
-      <mass value="15.0"/>
+      <mass value="5.0"/>
       <origin xyz="0.0 0 0.1" rpy=" 0 0 0"/>
       <inertia
@@ -33,5 +33,5 @@
         <sphere radius="0.05"/>
       </geometry>
-      <surface>
+      <!-- <surface>
         <friction>
           <ode>
@@ -42,5 +42,5 @@
           </ode>
         </friction>
-      </surface>
+      </surface> -->
     </collision>
     <visual name='caster_visual'>
@@ -55,5 +55,5 @@
         <sphere radius="0.05"/>
       </geometry>
-      <surface>
+      <!-- <surface>
         <friction>
           <ode>
@@ -64,5 +64,5 @@
           </ode>
         </friction>
-      </surface>
+      </surface> -->
     </collision>
     <visual name='caster_front_visual'>
@@ -127,5 +127,5 @@
     <parent link="chassis"/>
     <axis xyz="0 1 0" rpy="0 0 0"/>
-    <limit effort="10000" velocity="1000"/>
+    <!-- <limit effort="10000" velocity="1000"/> -->
     <joint_properties damping="0.0" friction="0.0"/>
   </joint>
@@ -136,8 +136,8 @@
     <parent link="chassis"/>
     <axis xyz="0 1 0" rpy="0 0 0"/>
-    <limit effort="10000" velocity="1000"/>
+    <!-- <limit effort="10000" velocity="1000"/> -->
     <joint_properties damping="0.0" friction="0.0"/>
   </joint>
-  <link name="camera">
+  <link name="camera_link">
     <collision>
       <origin xyz="0 0 0" rpy="0 0 0"/>
@@ -164,5 +164,5 @@
     <origin xyz=".2 0 0" rpy="0 0 0"/>
     <parent link="chassis"/>
-    <child link="camera"/>
+    <child link="camera_link"/>
   </joint>
   <!-- Hokuyo Laser -->
